File: nRF52832_MCU_Board/nRF52832_MCU_arduino/nRF52832_MCU.sch (EAGLE design)
At the start: 15 parts, among them U1 NRF52832, X1 32MHz

Commit message: Finished? footprint and symbol for nRF5, QFN. Done som experimenting on board layouts
Parts:
- removed U$1: 3.9nH, nRF:INDUCTOR(0402)
- added ANT1: 2.45GHZ_PCB_ANTENNA, nRF:2.45GHZ_PCB_ANTENNA
- added C13: 0.8pF, rcl:C-EUC0402
- added L1: 3.9nH, nRF:INDUCTOR(0402)
- added X2, X4: TSW-108-02-S-S, con-samtec:TSW-108-02-S-S
- added X3: TSW-106-02-S-S, con-samtec:TSW-106-02-S-S
- added X5: TSW-110-02-S-S, con-samtec:TSW-110-02-S-S
Connections:
- new net ANT: C3.1, L1.1, U1.ANT@30
- new net N$14: U1.SWDIO@26
- new net N$15: U1.SWDCLK@25
- new net P0.00: U1.P0.00/XL1@02, X3-6.1
- new net P0.01: U1.P0.01/XL2@03, X3-5.1
- new net P0.02: U1.P0.02/AIN0@04, X3-4.1
- new net P0.03: U1.P0.03/AIN1@05, X3-3.1
- new net P0.04: U1.P0.04/AIN2@06, X3-2.1
- new net P0.05: U1.P0.05/AIN3@07, X3-1.1
- new net P0.06: U1.P0.06@08, X4-8.1
- new net P0.07: U1.P0.07@09, X4-7.1
- new net P0.08: U1.P0.08@10, X4-6.1
- new net P0.09: U1.P0.09@11, X4-5.1
- new net P0.10: U1.P0.10@12, X4-4.1
- new net P0.11: U1.P0.11@14, X4-3.1
- new net P0.12: U1.P0.12@15, X4-2.1
- new net P0.13: U1.P0.13@16, X4-1.1
- new net P0.14: U1.P0.14@17, X5-10.1
- new net P0.15: U1.P0.15@18, X5-9.1
- new net P0.16: U1.P0.16@19, X5-8.1
- new net P0.17: U1.P0.17@20, X5-7.1
- new net P0.18: U1.P0.18@21, X5-6.1
- new net P0.19: U1.P0.19@22, X5-5.1
- new net P0.20: U1.P0.20@23, X5-3.1
- new net P0.21: U1.P0.21/RESET@24, X5-2.1
- new net P0.22: U1.P0.22@27, X5-1.1
- new net P0.23: U1.P0.23@28
- new net P0.24: U1.P0.24@29
- new net P0.25: U1.P0.25@37
- new net P0.26: U1.P0.26@38
- new net P0.27: U1.P0.27@39
- new net P0.28: U1.P0.28@40
- new net P0.29: U1.P0.29@41
- new net P0.30: U1.P0.30@42
- new net P0.31: U1.P0.31@43
- net GND: now also C13.2, X5-4.1
- net N$1: now also ANT1.P$1, C13.1, L1.2; no longer C3.1, U$1.1, U1.ANT@30
- net VCC: now also X2-2.1, X2-4.1, X2-5.1

Commit message: Copyed layout from nano to arduino
Parts:
- removed ANT1: 2.45GHZ_PCB_ANTENNA, nRF:2.45GHZ_PCB_ANTENNA
- removed X5: TSW-110-02-S-S, con-samtec:TSW-110-02-S-S
- added BATT1: CR1632, Nordic_misc:CR1632
- added C14, C15: 300pF, Nordic_misc:CAPACITOR_0402_N
- added C16: 100nF, Nordic_misc:CAPACITOR_0402_N
- added C17, C18: 10µF, Nordic_misc:CAPACITOR_0603_N
- added C19: 100µF, Nordic_misc:CAPACITOR_0805_N
- added C20: TBD, Nordic_misc:CAPACITOR_0402_N
- added D1, D2, D3: LED, Nordic_misc:LED
- added J5: MICROUSB, Nordic_misc:MICROUSB
- added J6: DEBUG_CONNECTOR, Nordic_misc:DEBUG_CONNECTOR
- added J7: FPC_05P-RA-SMD, Nordic_misc:FPC_05P-RA-SMD
- added J8: MM8130-2600, Nordic_misc:MM8130-2600
- added L2: 10µH, Nordic_misc:INDUCTOR_0603_N
- added L3: 15nH, Nordic_misc:INDUCTOR_0402_N
- added R1, R12, R2, R3, R4, U$6: 0R, Nordic_misc:RESISTOR_0402_N
- added R10, R11, R5, R6, R9: 330R, Nordic_misc:RESISTOR_0402_N
- added R7, R8: 100k, Nordic_misc:RESISTOR_0402_N
- added U$4, U$5: PANASONIC_EVQPT5A15, Nordic_misc:PANASONIC_EVQPT5A15
- added U2: TLV1117, Nordic_misc:TLV1117
- C1, C11, C12, C2, C3, C4, C5, C6, C7, C8: device rcl:C-EUC0402 -> Nordic_misc:CAPACITOR_0402_N
- C10, C9: device rcl:C-EUC0603 -> Nordic_misc:CAPACITOR_0603_N
- C13: value 0.8pF -> N.C.; device rcl:C-EUC0402 -> Nordic_misc:CAPACITOR_0402_N
- L1: device nRF:INDUCTOR(0402) -> Nordic_misc:INDUCTOR_0402_N
- U1: device nRF:NRF52832 -> Nordic_nRF:NRF52832
- X1: device IQD-Frequency-Products:CRYSTALS-GND-LID-IQXC-42 -> Nordic_nRF:XTAL_32MHZ
- X2: value TSW-108-02-S-S -> 32.768kHz; device con-samtec:TSW-108-02-S-S -> Nordic_nRF:XTAL_32KHZ
- X3: value TSW-106-02-S-S -> TSW-102-02-S-S-RA; device con-samtec:TSW-106-02-S-S -> con-samtec:TSW-102-02-S-S-RA
- X4: value TSW-108-02-S-S -> TSW-102-02-S-S-RA; device con-samtec:TSW-108-02-S-S -> con-samtec:TSW-102-02-S-S-RA
Connections:
- net N$4 renamed X1
- removed net N$14: U1.SWDIO@26
- removed net N$15: U1.SWDCLK@25
- removed net P0.18: U1.P0.18@21, X5-6.1
- removed net P0.21: U1.P0.21/RESET@24, X5-2.1
- removed net VCC: C5.1, C8.1, C9.1, U1.VDD@13, U1.VDD@36, U1.VDD@48, X2-2.1, X2-4.1, X2-5.1
- new net N$2: L2.2, L3.1
- new net N$4: L2.1, U1.DCC@47
- new net N$5: C13.1, J8.@IN, L1.2
- new net N$6: R6.2, R8.1, U$5.A, U$5.A'
- new net N$7: R5.2, R7.1, U$4.A, U$4.A'
- new net N$8: D2.C, R10.2
- new net N$9: D3.C, R11.2
- new net NFC1: C14.2, J7.2, R3.1, U1.P0.09/NFC1@11
- new net NFC2: C15.1, J7.4, R4.2, U1.P0.10/NFC2@12
- new net P0.18/SWO: J6.10, U1.P0.18/SWO@21
- new net P0.21/RESET: J6.6, R6.1, U1.P0.21/RESET@24
- new net SWDCLK: J6.4, U1.SWDCLK@25
- new net SWDIO: J6.2, U1.SWDIO@26
- new net VCC_P5V0_USB: J5.VBUS, R12.1
- new net VDD_LED: D1.A, R9.2
- new net VDD_P3V3: C18.1, C19.1, C5.1, C8.1, C9.1, D2.A, D3.A, J6.1, R7.2, R8.2, U$6.2, U1.VDD@13, U1.VDD@36, U1.VDD@48, U2.OUT
- new net VDD_P3V3_BATT: BATT1.+, U$6.1
- new net VDD_P5V0: C16.1, C17.1, D1.C, R12.2, U2.IN
- new net XL1: C11.2, R1.1, U1.P0.00/XL1@02, X2.1
- new net XL2: C12.2, R2.2, U1.P0.01/XL2@03, X2.2
- net DEC4: now also L3.2
- net GND: now also BATT1.-, C11.1, C12.1, C14.1, C15.2, C16.2, C17.2, C18.2, C19.2, C20.2, J5.GND, J6.3, J6.5, J6.9, J8.@GND, R9.1, U$4.B, U$4.B', U$4.GND, U$5.B, U$5.B', U$5.GND, U2.GND; no longer X5-4.1
- net N$1: now also C20.1, J8.@OUT; no longer ANT1.P$1, C13.1, L1.2
- net P0.00: now also R1.2; no longer U1.P0.00/XL1@02, X3-6.1
- net P0.01: now also R2.1; no longer U1.P0.01/XL2@03, X3-5.1
- net P0.02: no longer X3-4.1
- net P0.03: no longer X3-3.1
- net P0.04: no longer X3-2.1
- net P0.05: no longer X3-1.1
- net P0.06: now also R11.1; no longer X4-8.1
- net P0.07: now also R10.1; no longer X4-7.1
- net P0.08: now also R5.1; no longer X4-6.1
- net P0.09: now also R3.2; no longer U1.P0.09@11, X4-5.1
- net P0.10: now also R4.1; no longer U1.P0.10@12, X4-4.1
- net P0.11: no longer X4-3.1
- net P0.12: no longer X4-2.1
- net P0.13: no longer X4-1.1
- net P0.14: no longer X5-10.1
- net P0.15: no longer X5-9.1
- net P0.16: no longer X5-8.1
- net P0.17: no longer X5-7.1
- net P0.19: no longer X5-5.1
- net P0.20: no longer X5-3.1
- net P0.22: no longer X5-1.1
Other:
- note added: "Power supply"
