File: nRF52832_MCU_Board/nRF52832_MCU_nano/nRF52832_MCU.sch (EAGLE design)
At the start: 55 parts, among them J1 TSW-116-02-S-S, J2 TSW-116-02-S-S, J3 MM8130-2600, J4 FPC_05P-RA-SMD, J5 DEBUG_CONNECTOR, U1 NRF52832, X1 32MHz, X2 32.768kHz, X3 TSW-102-02-S-S-RA, X4 TSW-102-02-S-S-RA, X5 TSW-103-02-S-S, X6 TSW-103-02-S-S

Commit message: Fixed library links
Parts:
- ANT1: device nRF:ANTENNA_QUARTER-WAVE_MONOPOLE_MEANDERED_LEFT -> Nordic_misc:ANTENNA_QUARTER-WAVE_MONOPOLE_MEANDERED_LEFT
- C1, C11, C12, C13, C14, C15, C16, C2, C20, C3, C4, C5, C6, C7, C8: device nRF:CAPACITOR_0402_N -> Nordic_misc:CAPACITOR_0402_N
- C10, C17, C18, C9: device nRF:CAPACITOR_0603_N -> Nordic_misc:CAPACITOR_0603_N
- C19: device nRF:CAPACITOR_0805_N -> Nordic_misc:CAPACITOR_0805_N
- D1, D2, D3: device nRF:LED -> Nordic_misc:LED
- J3: device nRF:MM8130-2600 -> Nordic_misc:MM8130-2600
- J4: device nRF:FPC_05P-RA-SMD -> Nordic_misc:FPC_05P-RA-SMD
- J5: device nRF:DEBUG_CONNECTOR -> Nordic_misc:DEBUG_CONNECTOR
- L1, L3: device nRF:INDUCTOR_0402_N -> Nordic_misc:INDUCTOR_0402_N
- L2: device nRF:INDUCTOR_0603_N -> Nordic_misc:INDUCTOR_0603_N
- R1, R10, R11, R2, R3, R4, R5, R6, R7, R8, R9: device nRF:RESISTOR_0402_N -> Nordic_misc:RESISTOR_0402_N
- U$1: device nRF:MICROUSB -> Nordic_misc:MICROUSB
- U$2: device nRF:TLV1117 -> Nordic_misc:TLV1117
- U$3: device nRF:CR1632 -> Nordic_misc:CR1632
- U$4, U$5: device nRF:PANASONIC_EVQPT5A15 -> Nordic_misc:PANASONIC_EVQPT5A15
- U1: device nRF:NRF52832 -> Nordic_nRF:NRF52832
- X1: device nRF:XTAL_32MHZ -> Nordic_nRF:XTAL_32MHZ
- X2: device nRF:XTAL_32KHZ -> Nordic_nRF:XTAL_32KHZ

Commit message: Done some layout
Parts:
- added R12: 0R, Nordic_misc:RESISTOR_0402_N
Connections:
- removed net VCC: R7.2, R8.2
- removed net VCC_P3V3: C18.1, C19.1, C5.1, C8.1, C9.1, J5.1, U$2.OUT, U1.VDD@13, U1.VDD@36, U1.VDD@48, X5-2.1, X6-2.1
- removed net VCC_P5V0: C16.1, C17.1, U$2.IN, X5-1.1, X6-1.1
- new net N$8: D2.C, R10.2
- new net N$9: D3.C, R11.2
- new net VDD_LED: D1.A, R9.2
- new net VDD_P3V3: C18.1, C19.1, C5.1, C8.1, C9.1, D2.A, D3.A, J5.1, R7.2, R8.2, U$2.OUT, U1.VDD@13, U1.VDD@36, U1.VDD@48, X5-2.1, X6-2.1
- new net VDD_P5V0: C16.1, C17.1, D1.C, R12.2, U$2.IN, X5-1.1, X6-1.1
- net GND: now also R9.1
- net P0.06: now also R11.1
- net P0.07: now also R10.1
- net P0.08: now also R5.1
- net P0.21/RESET: now also R6.1
- net VCC_P5V0_USB: now also R12.1
Other:
- moved on the sheet: D1, D2, D3, R10, R11, R9, U$3

Commit message: Connected all signals in layout
Parts:
- removed U$1: MICROUSB, Nordic_misc:MICROUSB
- removed U$3: CR1632, Nordic_misc:CR1632
- removed X5, X6: TSW-103-02-S-S, con-samtec:TSW-103-02-S-S
- added BATT1: CR1632, Nordic_misc:CR1632
- added J6: DEBUG_CONNECTOR, Nordic_misc:DEBUG_CONNECTOR
- added J7: FPC_05P-RA-SMD, Nordic_misc:FPC_05P-RA-SMD
- added J8: MM8130-2600, Nordic_misc:MM8130-2600
- added U$6: 0R, Nordic_misc:RESISTOR_0402_N
- C13: value (none) -> N.C.
- C20: value (none) -> TBD
- J1: value TSW-116-02-S-S -> TSW-103-02-S-S; device con-samtec:TSW-116-02-S-S -> con-samtec:TSW-103-02-S-S
- J3: value MM8130-2600 -> TSW-116-02-S-S; device Nordic_misc:MM8130-2600 -> con-samtec:TSW-116-02-S-S
- J4: value FPC_05P-RA-SMD -> TSW-103-02-S-S; device Nordic_misc:FPC_05P-RA-SMD -> con-samtec:TSW-103-02-S-S
- J5: value DEBUG_CONNECTOR -> MICROUSB; device Nordic_misc:DEBUG_CONNECTOR -> Nordic_misc:MICROUSB
- renumbered U$2 to U2
Connections:
- new net VDD_P3V3_BATT: BATT1.+, U$6.1
- net GND: now also BATT1.-, J1-3.1, J4-3.1, J5.GND, J6.3, J6.5, J6.9, J8.@GND; no longer J3.@GND, J5.3, J5.5, J5.9, U$1.GND, X5-3.1, X6-3.1
- net N$1: now also J8.@OUT; no longer J3.@OUT
- net N$5: now also J8.@IN; no longer J3.@IN
- net NFC1: now also J7.2; no longer J4.2
- net NFC2: now also J7.4; no longer J4.4
- net P0.00: now also J3-9.1; no longer J2-9.1
- net P0.01: now also J3-8.1; no longer J2-8.1
- net P0.02: now also J3-7.1; no longer J2-7.1
- net P0.03: now also J3-6.1; no longer J2-6.1
- net P0.04: now also J3-5.1; no longer J2-5.1
- net P0.05: now also J3-4.1; no longer J2-4.1
- net P0.06: now also J3-3.1; no longer J2-3.1
- net P0.07: now also J3-2.1; no longer J2-2.1
- net P0.08: now also J3-1.1; no longer J2-1.1
- net P0.09: now also J2-1.1; no longer J1-1.1
- net P0.10: now also J2-2.1; no longer J1-2.1
- net P0.11: now also J2-3.1; no longer J1-3.1
- net P0.12: now also J2-4.1; no longer J1-4.1
- net P0.13: now also J2-5.1; no longer J1-5.1
- net P0.14: now also J2-6.1; no longer J1-6.1
- net P0.15: now also J2-7.1; no longer J1-7.1
- net P0.16: now also J2-8.1; no longer J1-8.1
- net P0.17: now also J2-9.1; no longer J1-9.1
- net P0.18/SWO: now also J2-10.1, J6.10; no longer J1-10.1, J5.10
- net P0.19: now also J2-11.1; no longer J1-11.1
- net P0.20: now also J2-12.1; no longer J1-12.1
- net P0.21/RESET: now also J2-13.1, J6.6; no longer J1-13.1, J5.6
- net P0.22: now also J2-14.1; no longer J1-14.1
- net P0.23: now also J2-15.1; no longer J1-15.1
- net P0.24: now also J2-16.1; no longer J1-16.1
- net P0.25: now also J3-16.1; no longer J2-16.1
- net P0.26: now also J3-15.1; no longer J2-15.1
- net P0.27: now also J3-14.1; no longer J2-14.1
- net P0.28: now also J3-13.1; no longer J2-13.1
- net P0.29: now also J3-12.1; no longer J2-12.1
- net P0.30: now also J3-11.1; no longer J2-11.1
- net P0.31: now also J3-10.1; no longer J2-10.1
- net SWDCLK: now also J6.4; no longer J5.4
- net SWDIO: now also J6.2; no longer J5.2
- net VCC_P5V0_USB: now also J5.VBUS; no longer U$1.VBUS
- net VDD_P3V3: now also J1-2.1, J4-2.1, J6.1, U$6.2; no longer J5.1, X5-2.1, X6-2.1
- net VDD_P5V0: now also J1-1.1, J4-1.1; no longer X5-1.1, X6-1.1
Other:
- moved on the sheet: J1-1, J1-2, J1-3, J2-1, J2-10, J2-11, J2-12, J2-13, J2-14, J2-15, J2-16, J2-2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

Commit message: Cleanup in layout
Parts:
- renumbered U$6 to R13
Other:
- moved on the sheet: C1, C2, X1
Changed lines of the file:
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@@
 <setting verticaltext="up"/>
 </settings>
-<grid distance="0.1" unitdist="inch" unit="inch" style="lines" multiple="1" display="yes" altdistance="0.01" altunitdist="inch" altunit="inch"/>
+<grid distance="0.1" unitdist="inch" unit="inch" style="lines" multiple="1" display="no" altdistance="0.01" altunitdist="inch" altunit="inch"/>
 <layers>
 <layer number="1" name="Top" color="4" fill="1" visible="no" active="no"/>
@@
 <part name="GND29" library="supply1" deviceset="GND" device=""/>
 <part name="VDD_NRF17" library="supply2" deviceset="VCC" device="" value="VDD_P3V3"/>
-<part name="U$6" library="Nordic_misc" deviceset="RESISTOR" device="_0402_N" value="0R"/>
+<part name="R13" library="Nordic_misc" deviceset="RESISTOR" device="_0402_N" value="0R"/>
 <part name="GND30" library="supply1" deviceset="GND" device=""/>
 <part name="VDD_P3V3_BATT" library="supply2" deviceset="VCC" device="" value="VDD_P3V3_BATT"/>
@@
 <instance part="VDD_NRF1" gate="G$1" x="83.82" y="139.7"/>
 <instance part="VDD_NRF2" gate="G$1" x="144.78" y="139.7"/>
-<instance part="GND10" gate="1" x="220.98" y="91.44" rot="MR0"/>
+<instance part="GND10" gate="1" x="226.06" y="104.14" rot="MR0"/>
 <instance part="GND11" gate="1" x="175.26" y="121.92" rot="MR0"/>
 <instance part="GND8" gate="1" x="228.6" y="71.12" rot="MR0"/>
-<instance part="X1" gate="X$1" x="205.74" y="101.6" rot="R90"/>
+<instance part="X1" gate="X$1" x="210.82" y="114.3" rot="R90"/>
 <instance part="ANT1" gate="G$1" x="241.3" y="86.36"/>
 <instance part="L1" gate="L$1" x="193.04" y="86.36" rot="R90"/>
 <instance part="L3" gate="L$1" x="104.14" y="149.86" rot="R180"/>
 <instance part="L2" gate="L$1" x="104.14" y="134.62" rot="R180"/>
-<instance part="C1" gate="C$1" x="213.36" y="114.3" rot="R90"/>
-<instance part="C2" gate="C$1" x="213.36" y="96.52" rot="R90"/>
+<instance part="C1" gate="C$1" x="218.44" y="127" rot="R90"/>
+<instance part="C2" gate="C$1" x="218.44" y="109.22" rot="R90"/>
 <instance part="C3" gate="C$1" x="182.88" y="81.28"/>
 <instance part="C4" gate="C$1" x="68.58" y="132.08"/>
@@
 <instance part="C10" gate="C$1" x="119.38" y="154.94"/>
 <instance part="C20" gate="C$1" x="228.6" y="81.28"/>
-<instance part="X2" gate="X$1" x="40.64" y="106.68" rot="R270"/>
+<instance part="X2" gate="X$1" x="40.64" y="106.68" smashed="yes" rot="R270">
+<attribute name="NAME" x="36.576" y="106.68" size="1.778" layer="95" rot="R270"/>
+<attribute name="VALUE" x="44.45" y="111.76" size="1.778" layer="96" rot="R270"/>
+</instance>
 <instance part="R1" gate="R$1" x="68.58" y="106.68" rot="R90"/>
 <instance part="R2" gate="R$1" x="68.58" y="88.9" rot="R90"/>
@@
 </segment>
 <segment>
-<wire x1="218.44" y1="114.3" x2="220.98" y2="114.3" width="0.1524" layer="91"/>
+<wire x1="223.52" y1="127" x2="226.06" y2="127" width="0.1524" layer="91"/>
 <pinref part="GND10" gate="1" pin="GND"/>
-<wire x1="220.98" y1="114.3" x2="220.98" y2="106.68" width="0.1524" layer="91"/>
-<wire x1="220.98" y1="106.68" x2="220.98" y2="104.14" width="0.1524" layer="91"/>
-<wire x1="220.98" y1="104.14" x2="220.98" y2="96.52" width="0.1524" layer="91"/>
-<wire x1="220.98" y1="96.52" x2="220.98" y2="93.98" width="0.1524" layer="91"/>
-<wire x1="218.44" y1="96.52" x2="220.98" y2="96.52" width="0.1524" layer="91"/>
-<junction x="220.98" y="96.52"/>
-<wire x1="208.28" y1="106.68" x2="220.98" y2="106.68" width="0.1524" layer="91"/>
-<junction x="220.98" y="106.68"/>
-<wire x1="208.28" y1="104.14" x2="220.98" y2="104.14" width="0.1524" layer="91"/>
-<junction x="220.98" y="104.14"/>
+<wire x1="226.06" y1="127" x2="226.06" y2="119.38" width="0.1524" layer="91"/>
+<wire x1="226.06" y1="119.38" x2="226.06" y2="116.84" width="0.1524" layer="91"/>
+<wire x1="226.06" y1="116.84" x2="226.06" y2="109.22" width="0.1524" layer="91"/>
+<wire x1="226.06" y1="109.22" x2="226.06" y2="106.68" width="0.1524" layer="91"/>
+<wire x1="223.52" y1="109.22" x2="226.06" y2="109.22" width="0.1524" layer="91"/>
+<junction x="226.06" y="109.22"/>
+<wire x1="213.36" y1="119.38" x2="226.06" y2="119.38" width="0.1524" layer="91"/>
+<junction x="226.06" y="119.38"/>
+<wire x1="213.36" y1="116.84" x2="226.06" y2="116.84" width="0.1524" layer="91"/>
+<junction x="226.06" y="116.84"/>
 <pinref part="X1" gate="X$1" pin="4"/>
 <pinref part="X1" gate="X$1" pin="2"/>
@@
 <net name="N$3" class="0">
 <segment>
-<wire x1="210.82" y1="114.3" x2="203.2" y2="114.3" width="0.1524" layer="91"/>
-<wire x1="203.2" y1="114.3" x2="203.2" y2="109.22" width="0.1524" layer="91"/>
-<wire x1="203.2" y1="114.3" x2="193.04" y2="114.3" width="0.1524" layer="91"/>
-<wire x1="193.04" y1="114.3" x2="193.04" y2="99.06" width="0.1524" layer="91"/>
-<junction x="203.2" y="114.3"/>
-<pinref part="U1" gate="U$1" pin="XC2@35"/>
-<wire x1="193.04" y1="99.06" x2="152.4" y2="99.06" width="0.1524" layer="91"/>
+<wire x1="215.9" y1="127" x2="208.28" y2="127" width="0.1524" layer="91"/>
+<wire x1="208.28" y1="127" x2="208.28" y2="121.92" width="0.1524" layer="91"/>
+<wire x1="208.28" y1="127" x2="198.12" y2="127" width="0.1524" layer="91"/>
+<wire x1="198.12" y1="127" x2="198.12" y2="111.76" width="0.1524" layer="91"/>
+<junction x="208.28" y="127"/>
 <pinref part="X1" gate="X$1" pin="3"/>
 <pinref part="C1" gate="C$1" pin="1"/>
+<pinref part="U1" gate="U$1" pin="XC2@35"/>
+<wire x1="198.12" y1="111.76" x2="198.12" y2="99.06" width="0.1524" layer="91"/>
+<wire x1="198.12" y1="99.06" x2="152.4" y2="99.06" width="0.1524" layer="91"/>
 </segment>
 </net>
 <net name="X1" class="0">
 <segment>
-<wire x1="203.2" y1="101.6" x2="203.2" y2="96.52" width="0.1524" layer="91"/>
-<wire x1="203.2" y1="96.52" x2="210.82" y2="96.52" width="0.1524" layer="91"/>
 <pinref part="U1" gate="U$1" pin="XC1@34"/>
-<wire x1="152.4" y1="96.52" x2="203.2" y2="96.52" width="0.1524" layer="91"/>
-<junction x="203.2" y="96.52"/>
+<wire x1="152.4" y1="96.52" x2="200.66" y2="96.52" width="0.1524" layer="91"/>
+<wire x1="200.66" y1="96.52" x2="200.66" y2="109.22" width="0.1524" layer="91"/>
+<pinref part="C2" gate="C$1" pin="1"/>
 <pinref part="X1" gate="X$1" pin="1"/>
-<pinref part="C2" gate="C$1" pin="1"/>
+<wire x1="208.28" y1="114.3" x2="208.28" y2="109.22" width="0.1524" layer="91"/>
+<wire x1="208.28" y1="109.22" x2="215.9" y2="109.22" width="0.1524" layer="91"/>
+<wire x1="200.66" y1="109.22" x2="208.28" y2="109.22" width="0.1524" layer="91"/>
+<junction x="208.28" y="109.22"/>
 </segment>
 </net>
@@
 <instance part="GND29" gate="1" x="104.14" y="38.1" rot="MR0"/>
 <instance part="VDD_NRF17" gate="G$1" x="144.78" y="106.68"/>
-<instance part="U$6" gate="R$1" x="134.62" y="104.14"/>
+<instance part="R13" gate="R$1" x="134.62" y="104.14"/>
 <instance part="GND30" gate="1" x="124.46" y="81.28" rot="MR0"/>
 <instance part="VDD_P3V3_BATT" gate="G$1" x="124.46" y="106.68"/>
@@
 </segment>
 <segment>
-<pinref part="U$6" gate="R$1" pin="2"/>
+<pinref part="R13" gate="R$1" pin="2"/>
 <pinref part="VDD_NRF17" gate="G$1" pin="VCC"/>
 <wire x1="139.7" y1="104.14" x2="144.78" y2="104.14" width="0.1524" layer="91"/>
@@
 <pinref part="BATT1" gate="G$1" pin="+"/>
 <wire x1="124.46" y1="101.6" x2="124.46" y2="104.14" width="0.1524" layer="91"/>
-<pinref part="U$6" gate="R$1" pin="1"/>
+<pinref part="R13" gate="R$1" pin="1"/>
 <wire x1="124.46" y1="104.14" x2="129.54" y2="104.14" width="0.1524" layer="91"/>
 <pinref part="VDD_P3V3_BATT" gate="G$1" pin="VCC"/>

Commit message: Added some vias
Connections:
- net N$6: no longer U$5.A'
Changed lines of the file:
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@@
 <net name="N$6" class="0">
 <segment>
-<pinref part="U$5" gate="G$1" pin="A'"/>
 <pinref part="R8" gate="R$1" pin="1"/>
-<wire x1="218.44" y1="134.62" x2="213.36" y2="134.62" width="0.1524" layer="91"/>
-<wire x1="213.36" y1="134.62" x2="213.36" y2="142.24" width="0.1524" layer="91"/>
 <pinref part="U$5" gate="G$1" pin="A"/>
 <wire x1="213.36" y1="142.24" x2="213.36" y2="144.78" width="0.1524" layer="91"/>
