File: nRF52832_MCU_Board/nRF52832_MCU_mini/nRF52832_MCU.brd (EAGLE design)
At the start: 45.7 x 22.9 mm, 19 parts, among them J1 TSW-116-02-S-S, J2 TSW-116-02-S-S, U1 NRF52832, X1 32MHz

Commit message: Finished? footprint and symbol for nRF5, QFN. Done som experimenting on board layouts
Parts:
- removed ANT1: 2.45GHZ_PCB_ANTENNA, nRF:PCB_ANTENNA
- removed J1, J2: TSW-116-02-S-S, con-samtec:TSW-116-02-S-S
- X1: device nRF:BT-XTAL_2016 -> IQD-Frequency-Products:2.0X1.6-4-PAD
- moved C13 15.6 mm to (1.50, -2.33)
- renumbered U1 to U$1
Connections:
- removed net N$14: U$1.26
- removed net N$15: U$1.25
- removed net P0.00: J1.1, U$1.2
- removed net P0.01: J1.2, U$1.3
- removed net P0.02: J1.3, U$1.4
- removed net P0.03: J1.4, U$1.5
- removed net P0.04: J1.5, U$1.6
- removed net P0.05: J1.6, U$1.7
- removed net P0.06: J1.7, U$1.8
- removed net P0.07: J1.8, U$1.9
- removed net P0.08: J1.9, U$1.10
- removed net P0.09: J1.10, U$1.11
- removed net P0.10: J1.11, U$1.12
- removed net P0.11: J1.12, U$1.14
- removed net P0.12: J1.13, U$1.15
- removed net P0.13: J1.14, U$1.16
- removed net P0.14: J1.15, U$1.17
- removed net P0.15: J1.16, U$1.18
- removed net P0.16: J2.16, U$1.19
- removed net P0.17: J2.15, U$1.20
- removed net P0.18: J2.14, U$1.21
- removed net P0.19: J2.13, U$1.22
- removed net P0.20: J2.12, U$1.23
- removed net P0.21: J2.11, U$1.24
- removed net P0.22: J2.10, U$1.27
- removed net P0.23: J2.9, U$1.28
- removed net P0.24: J2.8, U$1.29
- removed net P0.25: J2.7, U$1.37
- removed net P0.26: J2.6, U$1.38
- removed net P0.27: J2.5, U$1.39
- removed net P0.28: J2.4, U$1.40
- removed net P0.29: J2.3, U$1.41
- removed net P0.30: J2.2, U$1.42
- removed net P0.31: J2.1, U$1.43
- net ANT: no longer U$1.30
- net DEC2: no longer U$1.32
- net DEC3: no longer U$1.33
- net GND: now also X1.2, X1.4; no longer U$1.31, X1.P$2, X1.P$4
- net N$1: no longer ANT1.P$1
- net N$3: now also X1.3; no longer U$1.35, X1.P$3
- net N$4: now also X1.1; no longer U$1.34, X1.P$1
Routing:
- net GND: track 26.2 -> 3.29 mm
- net N$3: track 2.95 -> 6.42 mm

Commit message: Looked into different layout
Parts:
- removed C13: 0.8pF, rcl:C0402
- added L2: 10µH, Nordic_nRF:RESC0603_N
- added L3: 15nH, Nordic_nRF:RESC0402_N
- added U1: NRF52832, Nordic_nRF:QFN40P600X600X90-48_N
- added X2: 32.768kHz, Nordic_nRF:XTAL_3215_N
- added X3, X4: TSW-112-02-S-D, con-samtec:TSW-112-02-S-D
- added X5, X6: TSW-102-02-S-S-RA, con-samtec:TSW-102-02-S-S-RA
- C1, C11, C12, C2, C3, C4, C5, C6, C7, C8: device rcl:C0402 -> Nordic_nRF:RESC0402_N
- C10, C9: device rcl:C0603 -> Nordic_nRF:RESC0603_N
- L1: device nRF:R0402 -> Nordic_nRF:RESC0402_N
- U$1: value NRF52832 -> MICROUSB; device nRF:QFN40P600X600X90-48N -> Nordic_misc:USB-MICRO-B-RA-SMD-PIP
- X1: device IQD-Frequency-Products:2.0X1.6-4-PAD -> Nordic_nRF:BT-XTAL_2016_N
- moved U$1 34.1 mm to (-1.10, -0.40)
- moved C12 21.8 mm to (25.7, 27.9), turned to 270 degrees
- moved C11 21.7 mm to (25.7, 30.4), turned to 270 degrees
- moved C4 17.9 mm to (31.4, 27.4)
- moved C10 17.7 mm to (34.2, 30.3), turned to 90 degrees
- moved C9 17.7 mm to (31.4, 28.7)
- moved L1 16.6 mm to (42.8, 24.4)
- moved C3 16.5 mm to (41.2, 25.0)
- moved C5 16.5 mm to (33.0, 20.9)
- moved C6 16.2 mm to (41.8, 27.3)
- moved C7 16.1 mm to (41.8, 28.3)
- moved C8 16.0 mm to (38.8, 30.2)
- moved C1 16.0 mm to (39.8, 30.2)
- moved X1 16.0 mm to (41.8, 30.2)
- moved C2 15.9 mm to (43.8, 30.2)
Connections:
- removed net N$1: C13.1, L1.2
- removed net VCC: C5.1, C8.1, C9.1, U$1.13, U$1.36, U$1.48
- new net N$2: L2.2, L3.1
- new net P0.00/XL1: C11.2, U1.2, X2.1
- new net P0.01: U1.11
- new net P0.01/XL2: C12.2, U1.3, X2.2
- new net P0.02: U1.4
- new net P0.03: U1.5
- new net P0.04: U1.6
- new net P0.05: U1.7
- new net P0.06: U1.8
- new net P0.07: U1.9
- new net P0.08: U1.10
- new net P0.09: U1.12
- new net P0.11: U1.14
- new net P0.12: U1.15
- new net P0.13: U1.16
- new net P0.14: U1.17
- new net P0.15: U1.18
- new net P0.16: U1.19
- new net P0.17: U1.20
- new net P0.18/SWO: U1.21
- new net P0.19: U1.22
- new net P0.20: U1.23
- new net P0.21/RESET: U1.24
- new net P0.22: U1.27
- new net P0.23: U1.28
- new net P0.24: U1.29
- new net P0.25: U1.37
- new net P0.26: U1.38
- new net P0.27: U1.39
- new net P0.28: U1.40
- new net P0.29: U1.41
- new net P0.30: U1.42
- new net P0.31: U1.43
- new net RF: L1.2
- new net SWDCLK: U1.25
- new net SWDIO: U1.26
- new net VDD_P3V3: C5.1, C8.1, C9.1, U1.13, U1.36, U1.48
- new net X1: C2.1, U1.34, X1.1
- net ANT: now also U1.30
- net DEC1: now also U1.1; no longer U$1.1
- net DEC2: now also U1.32
- net DEC3: now also U1.33
- net DEC4: now also L3.2, U1.46; no longer U$1.46
- net GND: now also C11.1, C12.1, U1.31, U1.45, U1.PAD, U1.PAD@VIA01, U1.PAD@VIA02, U1.PAD@VIA03, U1.PAD@VIA04, U1.PAD@VIA05, U1.PAD@VIA06, U1.PAD@VIA07, U1.PAD@VIA08, U1.PAD@VIA09, U1.PAD@VIA10, U1.PAD@VIA11, U1.PAD@VIA12, U1.PAD@VIA13, U1.PAD@VIA14, U1.PAD@VIA15, U1.PAD@VIA16; no longer C13.2, U$1.45, U$1.PAD, U$1.PAD@VIA01, U$1.PAD@VIA02, U$1.PAD@VIA03, U$1.PAD@VIA04, U$1.PAD@VIA05, U$1.PAD@VIA06, U$1.PAD@VIA07, U$1.PAD@VIA08, U$1.PAD@VIA09, U$1.PAD@VIA10, U$1.PAD@VIA11, U$1.PAD@VIA12, U$1.PAD@VIA13, U$1.PAD@VIA14, U$1.PAD@VIA15, U$1.PAD@VIA16
- net N$3: now also U1.35
- net N$4: now also L2.1, U1.47; no longer C2.1, X1.1
Routing:
- net VDD_P3V3: track 0.00 -> 25.6 mm, vias 0 -> 3
- net GND: track 3.29 -> 26.9 mm, vias 0 -> 23
- net P0.00/XL1: track 0.00 -> 9.18 mm
- net X1: track 0.00 -> 8.06 mm
- net P0.01/XL2: track 0.00 -> 7.69 mm
- net P0.09: track 0.00 -> 7.50 mm
- net P0.08: track 0.00 -> 7.50 mm
- net P0.07: track 0.00 -> 7.50 mm
- net P0.06: track 0.00 -> 7.50 mm
- net P0.05: track 0.00 -> 7.50 mm
- net P0.04: track 0.00 -> 7.50 mm
- net P0.03: track 0.00 -> 7.50 mm
- net P0.02: track 0.00 -> 7.50 mm
- net P0.01: track 0.00 -> 7.50 mm
- net VCC: track 6.80 -> 0.00 mm
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Other:
- board size 45.7 x 22.9 mm -> 50 x 50 mm
