File: nRF52832_MCU_Board/nRF52832_MCU_mini/nRF52832_MCU.sch (EAGLE design)
At the start: 15 parts, among them U1 NRF52832, X1 32MHz

Commit message: Finished? footprint and symbol for nRF5, QFN. Done som experimenting on board layouts
Parts:
- removed U1: NRF52832, nRF:NRF52832
- added C13: 0.8pF, rcl:C-EUC0402
- added L1: 3.9nH, nRF:INDUCTOR(0402)
- U$1: value 3.9nH -> NRF52832; device nRF:INDUCTOR(0402) -> nRF:NRF52832
Connections:
- new net ANT: C3.1, L1.1
- net DEC1: now also U$1.DEC1@01; no longer U1.DEC1@01
- net DEC2: no longer U1.DEC2@32
- net DEC3: no longer U1.DEC3@33
- net DEC4: now also U$1.DEC4@46; no longer U1.DEC4@46
- net GND: now also C13.2, U$1.VSS@45; no longer U1.VSS@31, U1.VSS@45
- net N$1: now also C13.1, L1.2; no longer C3.1, U$1.1, U1.ANT@30
- net N$3: no longer U1.XC2@35
- net N$4: no longer U1.XC1@34
- net VCC: now also U$1.VDD@13, U$1.VDD@36, U$1.VDD@48; no longer U1.VDD@13, U1.VDD@36, U1.VDD@48
Other:
- moved on the sheet: C6, C7, C8

Commit message: Looked into different layout
Parts:
- removed C13: 0.8pF, rcl:C-EUC0402
- added L2: 10µH, Nordic_nRF:INDUCTOR_0603_N
- added L3: 15nH, Nordic_nRF:INDUCTOR_0402_N
- added U1: NRF52832, Nordic_nRF:NRF52832
- added X2: 32.768kHz, Nordic_nRF:XTAL_32KHZ
- added X3, X4: TSW-112-02-S-D, con-samtec:TSW-112-02-S-D
- added X5, X6: TSW-102-02-S-S-RA, con-samtec:TSW-102-02-S-S-RA
- C1, C11, C12, C2, C3, C4, C5, C6, C7, C8: device rcl:C-EUC0402 -> Nordic_nRF:CAPACITOR_0402_N
- C10, C9: device rcl:C-EUC0603 -> Nordic_nRF:CAPACITOR_0603_N
- L1: device nRF:INDUCTOR(0402) -> Nordic_nRF:INDUCTOR_0402_N
- U$1: value NRF52832 -> MICROUSB; device nRF:NRF52832 -> Nordic_misc:MICROUSB
- X1: device IQD-Frequency-Products:CRYSTALS-GND-LID-IQXC-42 -> Nordic_nRF:XTAL_32MHZ
Connections:
- removed net N$1: C13.1, L1.2
- removed net VCC: C5.1, C8.1, C9.1, U$1.VDD@13, U$1.VDD@36, U$1.VDD@48
- new net N$2: L2.2, L3.1
- new net P0.00/XL1: C11.2, U1.P0.00/XL1@02, X2.1
- new net P0.01: U1.P0.09/NFC1@11
- new net P0.01/XL2: C12.2, U1.P0.01/XL2@03, X2.2
- new net P0.02: U1.P0.02/AIN0@04
- new net P0.03: U1.P0.03/AIN1@05
- new net P0.04: U1.P0.04/AIN2@06
- new net P0.05: U1.P0.05/AIN3@07
- new net P0.06: U1.P0.06@08
- new net P0.07: U1.P0.07@09
- new net P0.08: U1.P0.08@10
- new net P0.09: U1.P0.10/NFC2@12
- new net P0.11: U1.P0.11@14
- new net P0.12: U1.P0.12@15
- new net P0.13: U1.P0.13@16
- new net P0.14: U1.P0.14@17
- new net P0.15: U1.P0.15@18
- new net P0.16: U1.P0.16@19
- new net P0.17: U1.P0.17@20
- new net P0.18/SWO: U1.P0.18/SWO@21
- new net P0.19: U1.P0.19@22
- new net P0.20: U1.P0.20@23
- new net P0.21/RESET: U1.P0.21/RESET@24
- new net P0.22: U1.P0.22@27
- new net P0.23: U1.P0.23@28
- new net P0.24: U1.P0.24@29
- new net P0.25: U1.P0.25@37
- new net P0.26: U1.P0.26@38
- new net P0.27: U1.P0.27@39
- new net P0.28: U1.P0.28@40
- new net P0.29: U1.P0.29@41
- new net P0.30: U1.P0.30@42
- new net P0.31: U1.P0.31@43
- new net RF: L1.2
- new net SWDCLK: U1.SWDCLK@25
- new net SWDIO: U1.SWDIO@26
- new net VDD_P3V3: C5.1, C8.1, C9.1, U1.VDD@13, U1.VDD@36, U1.VDD@48
- new net X1: C2.1, U1.XC1@34, X1.1
- net ANT: now also U1.ANT@30
- net DEC1: now also U1.DEC1@01; no longer U$1.DEC1@01
- net DEC2: now also U1.DEC2@32
- net DEC3: now also U1.DEC3@33
- net DEC4: now also L3.2, U1.DEC4@46; no longer U$1.DEC4@46
- net GND: now also C11.1, C12.1, U1.VSS@31, U1.VSS@45; no longer C13.2, U$1.VSS@45
- net N$3: now also U1.XC2@35
- net N$4: now also L2.1, U1.DCC@47; no longer C2.1, X1.1
