File: nRF52832_MCU_Board/nRF52832_MCU.brd (EAGLE design)
At the start: 55.7 x 22.9 mm, 55 parts, among them J1 TSW-103-02-S-S, J2 TSW-116-02-S-S, J3 TSW-116-02-S-S, J4 TSW-103-02-S-S, J5 MICROUSB, J6 DEBUG_CONNECTOR, J7 FPC_05P-RA-SMD, J8 MM8130-2600, U1 NRF52832, U2 TLV1117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

Commit message: Restructured MCU_Board
Parts:
- renumbered U$4 to BNT2, U$5 to BTN1
Changed lines of the file:
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@@
 </element>
 <element name="BATT1" library="Nordic_misc" package="CR1632_HOLDER_TH" value="CR1632" x="8.89" y="11.43" rot="MR270"/>
-<element name="U$4" library="Nordic_misc" package="PANASONIC_EVQPT5A15" value="PANASONIC_EVQPT5A15" x="18" y="15" smashed="yes"/>
-<element name="U$5" library="Nordic_misc" package="PANASONIC_EVQPT5A15" value="PANASONIC_EVQPT5A15" x="18" y="8" smashed="yes"/>
+<element name="BNT2" library="Nordic_misc" package="PANASONIC_EVQPT5A15" value="PANASONIC_EVQPT5A15" x="18" y="15" smashed="yes"/>
+<element name="BTN1" library="Nordic_misc" package="PANASONIC_EVQPT5A15" value="PANASONIC_EVQPT5A15" x="18" y="8" smashed="yes"/>
 <element name="R7" library="Nordic_misc" package="RESC0402_N" value="100k" x="14.3" y="13.4" smashed="yes" rot="R270">
 <attribute name="NAME" x="14.6" y="12.9" size="0.6" layer="25" rot="R90"/>
@@
 <wire x1="32.74" y1="5.55" x2="33.39" y2="5.55" width="0.2" layer="1"/>
 <wire x1="33.39" y1="5.55" x2="33.44" y2="5.6" width="0.2" layer="1"/>
-<contactref element="U$4" pad="6"/>
-<contactref element="U$4" pad="5"/>
-<contactref element="U$4" pad="3"/>
-<contactref element="U$4" pad="4"/>
-<contactref element="U$5" pad="6"/>
-<contactref element="U$5" pad="5"/>
-<contactref element="U$5" pad="3"/>
-<contactref element="U$5" pad="4"/>
+<contactref element="BNT2" pad="6"/>
+<contactref element="BNT2" pad="5"/>
+<contactref element="BNT2" pad="3"/>
+<contactref element="BNT2" pad="4"/>
+<contactref element="BTN1" pad="6"/>
+<contactref element="BTN1" pad="5"/>
+<contactref element="BTN1" pad="3"/>
+<contactref element="BTN1" pad="4"/>
 <via x="37.8" y="3.7" extent="1-16" drill="0.4"/>
 <contactref element="R9" pad="1"/>
@@
 <signal name="N$6">
 <contactref element="R8" pad="1"/>
-<contactref element="U$5" pad="1"/>
+<contactref element="BTN1" pad="1"/>
 <contactref element="R6" pad="2"/>
 <wire x1="14.3" y1="9.05" x2="15.45" y2="10.2" width="0.2" layer="1"/>
@@
 </signal>
 <signal name="N$7">
-<contactref element="U$4" pad="2"/>
+<contactref element="BNT2" pad="2"/>
 <contactref element="R7" pad="1"/>
-<contactref element="U$4" pad="1"/>
+<contactref element="BNT2" pad="1"/>
 <contactref element="R5" pad="2"/>
 <wire x1="14.3" y1="15.95" x2="14.3" y2="13.95" width="0.2" layer="1"/>

Commit message: Updated silk on some components, fixed via clearance at NFC and decoupling, fixed clearance at batt, routed XL1 and XL2, tented vias
Parts:
- moved C14 0.50 mm to (32.2, 8.20)
- moved C15 0.50 mm to (32.2, 6.10)
- moved R3 0.50 mm to (31.2, 8.20)
- moved R4 0.50 mm to (31.2, 6.10)
- moved C9 0.20 mm to (32.5, 15.1)
- moved L2 0.20 mm to (32.5, 16.6)
- moved L3 0.20 mm to (32.5, 17.9)
Routing:
- net NFC2: track 10.3 -> 10.9 mm
- net X1: track 7.46 -> 8.06 mm
- net P0.10: track 19.5 -> 19.0 mm
- net P0.09: track 24.6 -> 24.1 mm

Commit message: Done some work in silk
Parts:
- removed BNT2: PANASONIC_EVQPT5A15, Nordic_misc:PANASONIC_EVQPT5A15
- removed J1, J4: TSW-103-02-S-S, con-samtec:TSW-103-02-S-S
- removed J2, J3: TSW-116-02-S-S, con-samtec:TSW-116-02-S-S
- added BTN2: PANASONIC_EVQPT5A15, Nordic_misc:PANASONIC_EVQPT5A15
- added U$1, U$2: HEADER_3X1, Nordic_misc:HDRV3W64P254_1X3_762X254X900B_NO_SILK
- added U$3, U$4: HEADER_16X1, Nordic_misc:HDRV16W64P254_1X16_4064X254X900B_NO_SILK
- moved BTN1 7.00 mm to (18.0, 15.0)
Connections:
- net GND: now also BTN2.3, BTN2.4, BTN2.5, BTN2.6, U$1.P$1, U$2.P$3; no longer BNT2.3, BNT2.4, BNT2.5, BNT2.6, J1.3, J4.3
- net N$6: now also BTN2.1; no longer BTN1.1
- net N$7: now also BTN1.1, BTN1.2; no longer BNT2.1, BNT2.2
- net P0.00: now also U$4.P$8; no longer J3.9
- net P0.01: now also U$4.P$9; no longer J3.8
- net P0.02: now also U$4.P$10; no longer J3.7
- net P0.03: now also U$4.P$11; no longer J3.6
- net P0.04: now also U$4.P$12; no longer J3.5
- net P0.05: now also U$4.P$13; no longer J3.4
- net P0.06: now also U$4.P$14; no longer J3.3
- net P0.07: now also U$4.P$15; no longer J3.2
- net P0.08: now also U$4.P$16; no longer J3.1
- net P0.09: now also U$3.P$1; no longer J2.1
- net P0.10: now also U$3.P$2; no longer J2.2
- net P0.11: now also U$3.P$3; no longer J2.3
- net P0.12: now also U$3.P$4; no longer J2.4
- net P0.13: now also U$3.P$5; no longer J2.5
- net P0.14: now also U$3.P$6; no longer J2.6
- net P0.15: now also U$3.P$7; no longer J2.7
- net P0.16: now also U$3.P$8; no longer J2.8
- net P0.17: now also U$3.P$9; no longer J2.9
- net P0.18/SWO: now also U$3.P$10; no longer J2.10
- net P0.19: now also U$3.P$11; no longer J2.11
- net P0.20: now also U$3.P$12; no longer J2.12
- net P0.21/RESET: now also U$3.P$13; no longer J2.13
- net P0.22: now also U$3.P$14; no longer J2.14
- net P0.23: now also U$3.P$15; no longer J2.15
- net P0.24: now also U$3.P$16; no longer J2.16
- net P0.25: now also U$4.P$1; no longer J3.16
- net P0.26: now also U$4.P$2; no longer J3.15
- net P0.27: now also U$4.P$3; no longer J3.14
- net P0.28: now also U$4.P$4; no longer J3.13
- net P0.29: now also U$4.P$5; no longer J3.12
- net P0.30: now also U$4.P$6; no longer J3.11
- net P0.31: now also U$4.P$7; no longer J3.10
- net VDD_P3V3: now also U$1.P$2, U$2.P$2; no longer J1.2, J4.2
- net VDD_P5V0: now also U$1.P$3, U$2.P$1; no longer J1.1, J4.1
Routing:
- net P0.06: track 30.6 -> 28.8 mm, vias 1 -> 2
- net P0.21/RESET: track 45.5 -> 44.2 mm, vias 1 -> 2
- net VDD_P5V0: track 68.1 -> 67.2 mm
- net P0.07: track 33.1 -> 33.5 mm, vias 1 -> 2
Other:
- board text added: "00"
- board text added: "01"
- board text added: "02"
- board text added: "03"
- board text added: "04"
- board text added: "05"
- board text added: "06"
- board text added: "07"
- board text added: "08"
- board text added: "09"
- board text added: "10"
- board text added: "11"
- board text added: "12"
- board text added: "13"
- board text added: "14"
- board text added: "15"
- board text added: "16"
- board text added: "17"
- board text added: "18"
- board text added: "19"
- board text added: "20"
- board text added: "21"
- board text added: "22"
- board text added: "23"
- board text added: "24"
- board text added: "25"
- board text added: "26"
- board text added: "27"
- board text added: "28"
- board text added: "29"
- board text added: "30"
- board text added: "31"
- board text added: "3V3"
- board text added: "4"
- board text added: "5"
- board text added: "5V0"
- board text added: "BTN1"
- board text added: "CR1632"
- board text added: "GND"
- board text added: "J5"
- board text added: "J6"
- board text added: "J7"
- board text added: "J8"
- board text added: "LED1"
- board text added: "LED2"
- board text added: "NFCT"
- board text added: "PWR"
- board text added: "RESET"
- board text added: "nRF52832"
- board text added: "nRF52832_MCU_Board"
