File: nRF52832_MCU_Board/nRF52832_MCU.brd (EAGLE design)
At the start: 55.7 x 22.9 mm, 55 parts, among them J5 MICROUSB, J6 DEBUG_CONNECTOR, J7 FPC_05P-RA-SMD, J8 MM8130-2600, U1 NRF52832, U2 TLV1117, X1 32MHz, X2 32.768kHz

Commit message: Added more vias, fixed error in silkscreen at J1
Routing:
- net GND: vias 76 -> 101

Commit message: Added name to headers in library, named headers properly
Parts:
- renumbered U$1 to J4, U$2 to J1, U$3 to J2, U$4 to J3
