File: nRF52832_reference/nRF52832_qfaa_nfc/nRF52832_qfaa_nfc.brd (EAGLE design)
At the start: 30 x 74 mm, 21 parts, among them U1 NRF52832, X1 32MHz, X2 32.768kHz

Commit message: Added more vias
Routing:
- net GND: vias 14 -> 24
Changed lines of the file:
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@@
 <contactref element="C13" pad="1"/>
 <contactref element="C14" pad="2"/>
-<wire x1="13.15" y1="62.9" x2="16.35" y2="62.9" width="0" layer="19" extent="1-1"/>
+<via x="10.9" y="73.1" extent="1-16" drill="0.4" diameter="0.8"/>
+<via x="14.8" y="73.1" extent="1-16" drill="0.4" diameter="0.8"/>
+<via x="29.1" y="73.1" extent="1-16" drill="0.4" diameter="0.8"/>
+<via x="26.7" y="63.7" extent="1-16" drill="0.4" diameter="0.8"/>
+<via x="29.1" y="60.9" extent="1-16" drill="0.4" diameter="0.8"/>
+<via x="26.7" y="60.9" extent="1-16" drill="0.4" diameter="0.8"/>
+<via x="16.4" y="61.9" extent="1-16" drill="0.4" diameter="0.8"/>
+<via x="10.9" y="60.9" extent="1-16" drill="0.4" diameter="0.8"/>
+<via x="10.9" y="63.8" extent="1-16" drill="0.4" diameter="0.8"/>
+<via x="13.1" y="63.9" extent="1-16" drill="0.4" diameter="0.8"/>
 </signal>
 <signal name="DEC1">

Commit message: Issue #2: Fixed value of C7 from 100nF to 100pF
Parts:
- C7: value 100nF -> 100pF
Changed lines of the file:
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@@
 <attribute name="VALUE" x="26.1" y="66.3" size="1.27" layer="27"/>
 </element>
-<element name="C7" library="Nordic_nRF" package="RESC0402_N" value="100nF" x="26.8" y="69.3" smashed="yes">
+<element name="C7" library="Nordic_nRF" package="RESC0402_N" value="100pF" x="26.8" y="69.3" smashed="yes">
 <attribute name="NAME" x="26.3" y="69" size="0.6" layer="25"/>
 <attribute name="VALUE" x="26.1" y="67.3" size="1.27" layer="27"/>

Commit message: Same fixes as in qfaa_dcdc
Parts:
- moved C1 4.00 mm to (28.8, 71.2), turned to 270 degrees
- moved C2 4.00 mm to (24.8, 71.2), turned to 90 degrees
Connections:
- net N$3: now also C2.1; no longer C1.1
- net X1: now also C1.1; no longer C2.1
Changed lines of the file:
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@@
 <?xml version="1.0" encoding="utf-8"?>
 <!DOCTYPE eagle SYSTEM "eagle.dtd">
-<eagle version="7.6.0">
+<eagle version="8.3.0">
 <drawing>
 <settings>
 <setting alwaysvectorfont="no"/>
+<setting keepoldvectorfont="yes"/>
 <setting verticaltext="up"/>
 </settings>
@@
 <attribute name="VALUE" x="27.1" y="63.45" size="1.27" layer="27"/>
 </element>
-<element name="C1" library="Nordic_nRF" package="RESC0402_N" value="12pF" x="24.8" y="71.2" smashed="yes" rot="R90">
+<element name="C2" library="Nordic_nRF" package="RESC0402_N" value="12pF" x="24.8" y="71.2" smashed="yes" rot="R90">
 <attribute name="NAME" x="25.1" y="70.7" size="0.6" layer="25" rot="R90"/>
 <attribute name="VALUE" x="26.8" y="70.5" size="1.27" layer="27" rot="R90"/>
 </element>
-<element name="C2" library="Nordic_nRF" package="RESC0402_N" value="12pF" x="28.8" y="71.2" smashed="yes" rot="R270">
+<element name="C1" library="Nordic_nRF" package="RESC0402_N" value="12pF" x="28.8" y="71.2" smashed="yes" rot="R270">
 <attribute name="NAME" x="29.1" y="70.7" size="0.6" layer="25" rot="R90"/>
 <attribute name="VALUE" x="26.8" y="71.9" size="1.27" layer="27" rot="R270"/>
@@
 <contactref element="X1" pad="4"/>
 <contactref element="X1" pad="2"/>
+<contactref element="C2" pad="2"/>
 <contactref element="C1" pad="2"/>
-<contactref element="C2" pad="2"/>
 <contactref element="C3" pad="2"/>
 <contactref element="C4" pad="2"/>
@@
 <contactref element="U1" pad="35"/>
 <contactref element="X1" pad="3"/>
-<contactref element="C1" pad="1"/>
+<contactref element="C2" pad="1"/>
 <wire x1="24" y1="67.8" x2="24.4" y2="67.8" width="0.2" layer="1"/>
 <wire x1="24.4" y1="67.8" x2="24.7" y2="68.1" width="0.2" layer="1"/>
@@
 <contactref element="U1" pad="34"/>
 <contactref element="X1" pad="1"/>
-<contactref element="C2" pad="1"/>
+<contactref element="C1" pad="1"/>
 <wire x1="28.8" y1="71.75" x2="27.55" y2="71.75" width="0.2" layer="1"/>
 <wire x1="27.55" y1="71.75" x2="27.525" y2="71.775" width="0.2" layer="1"/>
