File: nRF52810_reference/nRF52810_qfaa_dcdc/nRF52810_qfaa_dcdc.brd (EAGLE design)
At the start: 20 x 14 mm, 18 parts, among them U1 NRF52832, X1 32MHz, X2 32.768kHz

Commit message: Eagle did not save properly
Parts:
- U1: value NRF52832 -> NRF52810_QF
Changed lines of the file:
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@@
 </autorouter>
 <elements>
-<element name="U1" library="Nordic_nRF" package="QFN40P600X600X90-48_N" value="NRF52832" x="11" y="6" smashed="yes">
+<element name="U1" library="Nordic_nRF" package="QFN40P600X600X90-48_N" value="NRF52810_QF" x="11" y="6" smashed="yes">
 <attribute name="NAME" x="10.6" y="5.7" size="0.6" layer="25" ratio="11"/>
 <attribute name="VALUE" x="9" y="9.6" size="0.889" layer="27" ratio="11"/>
