File: nRF52810_reference/nRF52810_qfaa_dcdc/nRF52810_qfaa_dcdc.sch (EAGLE design)
At the start: 18 parts, among them U1 NRF52832, X1 32MHz, X2 32.768kHz

Commit message: Eagle did not save properly
Parts:
- U1: value NRF52832 -> NRF52810_QF; device Nordic_nRF:NRF52832 -> Nordic_nRF:NRF52810_QF
Connections:
- net DEC1: now also U1.DEC1@1; no longer U1.DEC1@01
- net P0.00/XL1: now also U1.P0.00/XL1@2; no longer U1.P0.00/XL1@02
- net P0.01/XL2: now also U1.P0.01/XL2@3; no longer U1.P0.01/XL2@03
- net P0.02: now also U1.P0.02/AIN0@4; no longer U1.P0.02/AIN0@04
- net P0.03: now also U1.P0.03/AIN1@5; no longer U1.P0.03/AIN1@05
- net P0.04: now also U1.P0.04/AIN2@6; no longer U1.P0.04/AIN2@06
- net P0.05: now also U1.P0.05/AIN3@7; no longer U1.P0.05/AIN3@07
- net P0.06: now also U1.P0.06@8; no longer U1.P0.06@08
- net P0.07: now also U1.P0.07@9; no longer U1.P0.07@09
- net P0.09: now also U1.P0.09@11; no longer U1.P0.09/NFC1@11
- net P0.10: now also U1.P0.10@12; no longer U1.P0.10/NFC2@12
- net P0.18/SWO: now also U1.P0.19@21; no longer U1.P0.18/SWO@21
- net P0.28: now also U1.P0.28/AIN4@40; no longer U1.P0.28@40
- net P0.29: now also U1.P0.29/AIN5@41; no longer U1.P0.29@41
- net P0.30: now also U1.P0.30/AIN6@42; no longer U1.P0.30@42
- net P0.31: now also U1.P031/AIN7@43; no longer U1.P0.31@43
